File: Hardware - KiCAD/KiCAD-Project/FSEI_Wuerfel.kicad_pcb (KiCad board)
At the start: 2 copper layers, 35 x 60 mm, 30 parts, among them SW1 SK12D07VG4, SW2 Omron B3F-4055, U1 ATtiny13A-P

Commit message: added interactive BOM
Parts:
- JP1: value SolderJumper_2_Open -> Close if R8 and C2 (LowPass Filter) is NOT populated
- JP2: value SolderJumper_2_Bridged -> Close if SW1 is NOT populated
Changed lines of the file:
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@@
         (effects (font (size 1 1) (thickness 0.15)))
     )
-    (fp_text value "SolderJumper_2_Open" (at 0 1.9 90) (layer "F.Fab") hide
+    (fp_text value "Close if R8 and C2 (LowPass Filter) is NOT populated" (at 0 1.9 90) (layer "F.Fab") hide
         (effects (font (size 1 1) (thickness 0.15)))
     )
@@
     (property "ki_description" "Solder Jumper, 2-pole, closed/bridged")
     (property "ki_keywords" "solder jumper SPST")
-    (attr exclude_from_pos_files exclude_from_bom)
+    (attr exclude_from_pos_files)
     (fp_text reference "JP2" (at 0 1.823609 180) (layer "F.SilkS")
         (effects (font (size 1 1) (thickness 0.15)))
     )
-    (fp_text value "SolderJumper_2_Bridged" (at 0 1.9 180) (layer "F.Fab") hide
-        (effects (font (size 1 1) (thickness 0.15)))
-    )
+    (fp_text value "Close if SW1 is NOT populated" (at 0 1.9 180) (layer "F.Fab") hide
+        (effects (font (size 1 1) (thickness 0.15)))
+    )
